Commit message: Added 4 pulley config

File: gz-simulator/src/pulley_package/urdf/pulley_motor.urdf (robot description, URDF)
Before this commit: robot pulley_system, 3 links, 2 joints
Links:
- removed link pulley
- removed link rope_attachment
- added link wall, mass 100.0; collision box size=${wall_width} ${wall_thickness} ${wall_height}; visual box size=${wall_width} ${wall_thickness} ${wall_height}
- added link world
- link base_link: mass 1.0 -> 0.001; geometry 
Joints:
- removed joint motor_joint
- removed joint rope_joint
- added joint wall_joint: type fixed, parent base_link, child wall, origin xyz=0 0 ${wall_height/2} rpy=0 0 0
- added joint world_joint: type fixed, parent world, child base_link, origin xyz=0 0 0 rpy=0 0 0
